Commit message: adding files

File: src/my_robot/urdf/my_robot.xacro (robot description, xacro)
@@ -118,4 +118,10 @@
     </inertial>
   </link>
+  <joint name="camera_optical_joint" type="fixed">
+    <origin xyz="0 0 0" rpy="-1.5707 0 -1.5707"/>
+    <parent link="camera_link"/>
+    <child link="camera_link_optical"/>
+  </joint>
+  <link name="camera_link_optical"></link>
   <joint type="fixed" name="camera_joint">
     <origin xyz="0.2 0 0" rpy="0 0 0"/>

Commit message: working on project

File: src/my_robot/urdf/my_robot.xacro (robot description, xacro)
@@ -126,5 +126,5 @@
   <joint type="fixed" name="camera_joint">
     <origin xyz="0.2 0 0" rpy="0 0 0"/>
-    <child link="camera"/>
+    <child link="camera_link"/>
     <parent link="chassis"/>
     <axis xyz="0 1 0" rpy="0 0 0"/>
@@ -132,5 +132,5 @@
     <dynamics damping="1.0" friction="1.0"/>
   </joint>
-   <link name="camera">
+   <link name="camera_link">
     <visual>
       <origin xyz="0.0 0.0 0.03" rpy="0 0 0"/>
